Commit message: attempting to get gazebo sim working

File: workspace/src/rookie_description/urdf/rookie.urdf (robot description, URDF)
Before this commit: robot rookie, 5 links, 4 joints
Links:
- added link camera; visual box size=0.01 0.05 0.01
- added link lidar_slamtec_c1; collision cylinder length=0.0413 radius=0.0278; visual cylinder length=0.0413 radius=0.0278
- link front_left_wheel: geometry collision cylinder length=0.02032 radius=0.0492125; visual mesh filename=/home/wfletcher/workspace/install/rookie_description/share/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
- link front_right_wheel: geometry collision cylinder length=0.02032 radius=0.0492125; visual mesh filename=/home/wfletcher/workspace/install/rookie_description/share/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
- link rear_left_wheel: geometry collision cylinder length=0.02032 radius=0.0492125; visual mesh filename=/home/wfletcher/workspace/install/rookie_description/share/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
- link rear_right_wheel: geometry collision cylinder length=0.02032 radius=0.0492125; visual mesh filename=/home/wfletcher/workspace/install/rookie_description/share/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
Joints:
- added joint camera_joint: type fixed, parent base_link, child camera, origin xyz=0.1130775 0 0 rpy=0.0 0.0 0
- added joint lidar_joint: type fixed, parent base_link, child lidar_slamtec_c1, origin xyz=0 0 0.06015 rpy=0.0 0.0 0

File: workspace/src/rookie_description/urdf/rookie.urdf.xacro (robot description, xacro)
@@ -18,4 +18,7 @@
     <xacro:property name="wheel_spacing" value="0.00546" />
     <xacro:property name="wheel_mass" value="0.0992233" />
+    <!-- Rather than deal with whatever URDF/SDF package-finding weirdness Gazebo has going on,
+         just get our mesh paths directly here so we can use them later.-->
+    <xacro:property name="mesh_directory" value="$(find rookie_description)/meshes/" />
     <!-- Macros -->
     <xacro:include filename="$(find rookie_description)/urdf/macros.xacro" />
@@ -59,5 +62,5 @@
             <origin rpy="0.0 0.0 0.0" xyz="0.0 0.0 0.0" />
             <geometry>
-                <mesh filename="package://rookie_description/meshes/Banebots_T81_Wheel.dae"/>
+                <mesh filename="${mesh_directory}/Banebots_T81_Wheel.dae"/>
             </geometry>
         </visual>
@@ -74,5 +77,5 @@
             <origin rpy="0.0 0.0 0.0" xyz="0.0 0.0 0.0" />
             <geometry>
-                <mesh filename="package://rookie_description/meshes/Banebots_T81_Wheel.dae"/>
+                <mesh filename="${mesh_directory}/Banebots_T81_Wheel.dae"/>
             </geometry>
         </visual>
@@ -89,5 +92,5 @@
             <origin rpy="0.0 0.0 0.0" xyz="0.0 0.0 0.0" />
             <geometry>
-                <mesh filename="package://rookie_description/meshes/Banebots_T81_Wheel.dae"/>
+                <mesh filename="${mesh_directory}/Banebots_T81_Wheel.dae"/>
             </geometry>
         </visual>
@@ -104,5 +107,5 @@
             <origin rpy="0.0 0.0 0.0" xyz="0.0 0.0 0.0" />
             <geometry>
-                <mesh filename="package://rookie_description/meshes/Banebots_T81_Wheel.dae"/>
+                <mesh filename="${mesh_directory}/Banebots_T81_Wheel.dae"/>
             </geometry>
         </visual>
@@ -115,3 +118,40 @@
         <xacro:wheel_joint wheel_name="rear_right_wheel" mirror_x="-1" mirror_y="-1" />
     </joint>
+    <link name="lidar_slamtec_c1">
+        <visual>
+            <origin rpy="0.0 0.0 0.0" xyz="0.0 0.0 0.0" />
+            <geometry>
+                <cylinder length="0.0413" radius="0.0278" />
+            </geometry>
+        </visual>
+        <collision>
+            <geometry>
+                <cylinder length="0.0413" radius="0.0278" />
+            </geometry>
+        </collision>
+    </link>
+    <joint name="lidar_joint" type="fixed">
+        <parent link="base_link" />
+        <child link="lidar_slamtec_c1" />
+        <origin
+            xyz="0 0 ${(base_height / 2) + (0.0413 / 2)}"
+            rpy="0.0 0.0 0"/>
+    </joint>
+    <link name="camera">
+        <static>true</static>
+        <visual name='visual'>
+            <geometry>
+                <box size="0.01 0.05 0.01" />
+            </geometry>
+        </visual>
+    </link>
+    <joint name="camera_joint" type="fixed">
+        <parent link="base_link" />
+        <child link="camera" />
+        <origin
+            xyz="${base_length / 2} 0 0"
+            rpy="0.0 0.0 0"/>
+    </joint>
+    <!-- Gazebo-specific -->
+    <xacro:include filename="$(find rookie_description)/urdf/rookie_gazebo.xacro" />
 </robot>

File: workspace/src/rookie_description/urdf/rookie_gazebo.xacro (robot description, xacro)
@@ -1,5 +1,86 @@
 <?xml version="1.0"?>
 <robot xmlns:xacro="http://www.ros.org/wiki/xacro">
+    <!-- The plugins we need to be loaded -->
     <gazebo>
+        <!-- plugin type "imu" -->
+        <plugin filename="gz-sim-imu-system" name="gz::sim::systems::Imu" />
+        <!-- LiDAR ('gpu_lidar') plugin, Camera ('camera') -->
+        <plugin filename="gz-sim-sensors-system" name="gz::sim::systems::Sensors" />
+    </gazebo>
+    <!-- "Global" sensors, not explicitly attached to any link -->
+    <gazebo>
+        <!-- Differential drive (skid steer) plugin -->
+        <plugin filename="gz-sim-diff-drive-system" name="gz::sim::systems::DiffDrive">
+            <update_rate>30</update_rate>
+            <left_joint>front_left_wheel_joint</left_joint>
+            <left_joint>rear_left_wheel_joint</left_joint>
+            <right_joint>front_right_wheel_joint</right_joint>
+            <right_joint>rear_right_wheel_joint</right_joint>
+            <wheel_separation>${track_width}</wheel_separation>
+            <wheel_radius>${wheel_diameter / 2}</wheel_radius>
+            <odom_publish_frequency>50</odom_publish_frequency>
+            <frame_id>odom</frame_id>
+            <topic>cmd_vel</topic>
+        </plugin>
+    </gazebo>
+    <!-- Sensors attached to the base_link -->
+    <gazebo reference="base_link">
+        <!-- IMU plugin -->
+        <sensor name="imu_sensor" type="imu">
+            <always_on>1</always_on>
+            <update_rate>20</update_rate>
+            <visualize>false</visualize>
+            <topic>imu</topic>
+        </sensor>
+    </gazebo>
+    <!-- Sensors attached to the lidar_slamtec_c1 link -->
+    <gazebo reference="lidar_slamtec_c1">
+        <sensor name="lidar_slamtec_c1_sensor" type="gpu_lidar">
+            <pose relative_to='lidar_joint'>0 0 0 0 0 0</pose>
+            <always_on>1</always_on>
+            <visualize>true</visualize>
+            <topic>lidar</topic>
+            <update_rate>10</update_rate>
+            <ray>
+                <scan>
+                    <horizontal>
+                        <samples>640</samples>
+                        <resolution>1</resolution>
+                        <min_angle>-1.396263</min_angle>
+                        <max_angle>1.396263</max_angle>
+                    </horizontal>
+                    <vertical>
+                        <samples>1</samples>
+                        <resolution>0.01</resolution>
+                        <min_angle>0</min_angle>
+                        <max_angle>0</max_angle>
+                    </vertical>
+                </scan>
+                <range>
+                    <min>0.08</min>
+                    <max>10.0</max>
+                    <resolution>0.01</resolution>
+                </range>
+            </ray>
+        </sensor>
+    </gazebo>
+    <gazebo reference="camera">
+        <sensor name="camera_sensor" type="camera">
+          <camera>
+            <horizontal_fov>1.047</horizontal_fov>
+            <image>
+              <width>320</width>
+              <height>240</height>
+            </image>
+            <clip>
+              <near>0.1</near>
+              <far>100</far>
+            </clip>
+          </camera>
+          <always_on>1</always_on>
+          <update_rate>30</update_rate>
+          <visualize>true</visualize>
+          <topic>camera</topic>
+        </sensor>
     </gazebo>
 </robot>
