Commit message: working tree

File: workspace/src/rookie_description/urdf/rookie.urdf.xacro (robot description, xacro)
@@ -1,15 +1,23 @@
 <?xml version="1.0"?>
 <robot name="rookie" xmlns:xacro="http://www.ros.org/wiki/xacro">
+    <!-- Wheelbase: center to center distance between front and back wheels -->
     <xacro:property name="wheel_base" value="0.129" />
+    <!-- Track width: center to center distance between left and right wheels -->
     <xacro:property name="track_width" value="0.204" />
+    <!-- Ground clearance: distance from bottom of chassis to the ground -->
     <xacro:property name="ground_clearance" value="0.020" /> <!-- approximate -->
-    <!-- Base link dimensions -->
+    <!-- Base dimensions -->
     <xacro:property name="base_length" value="0.226155" />
     <xacro:property name="base_width" value="0.147" />
     <xacro:property name="base_height" value="0.079" />
+    <xacro:property name="base_mass" value="2" /> <!-- just a guess -->
     <!-- Critical dimensions of the wheels-->
     <xacro:property name="wheel_width" value="0.02032" />
-    <xacro:property name="wheel_diameter" value="0.098425" /> <!-- 3 7/8" -->
-    <xacro:property name="wheel_spacing" value="0.00546" /> <!-- clearance between wheel and body -->
+    <xacro:property name="wheel_diameter" value="0.098425" /> <!-- == 3 7/8" -->
+    <!-- wheel spacing: clearance between wheel and body -->
+    <xacro:property name="wheel_spacing" value="0.00546" />
+    <xacro:property name="wheel_mass" value="0.0992233" />
+    <!-- Macros -->
+    <xacro:include filename="$(find rookie_description)/urdf/macros.xacro" />
     <xacro:macro name="wheel_dimensions">
         <origin xyz="0 ${-1 * wheel_width / 2} 0" rpy="1.570796327 0 0"/>
@@ -18,16 +26,4 @@
         </geometry>
     </xacro:macro>
-    <link name="base_link">
-        <visual>
-            <geometry>
-                <box size="${base_length} ${base_width} ${base_height}"/>
-            </geometry>
-        </visual>
-        <collision>
-            <geometry>
-                <box size="${base_length} ${base_width} ${base_height}"/>
-            </geometry>
-        </collision>
-    </link>
     <xacro:macro name="wheel_joint" params="wheel_name mirror_x mirror_y">
         <parent link="base_link" />
@@ -43,8 +39,20 @@
                  ${((track_width / 2) + wheel_spacing - (wheel_width / 2)) * mirror_y}
                  ${-(base_height / 2) - ground_clearance + (wheel_diameter / 2)}"
-            rpy="0.0
-                0.0
-                ${yaw}"/>
+            rpy="0.0 0.0 ${yaw}"/>
     </xacro:macro>
+    <!-- /Macros -->
+    <link name="base_link">
+        <visual>
+            <geometry>
+                <box size="${base_length} ${base_width} ${base_height}"/>
+            </geometry>
+        </visual>
+        <collision>
+            <geometry>
+                <box size="${base_length} ${base_width} ${base_height}"/>
+            </geometry>
+        </collision>
+        <xacro:box_inertia name="base_link" mass="2" width="${base_width}" height="${base_height}" length="${base_length}" />
+    </link>
     <link name="front_left_wheel">
         <visual>
@@ -57,4 +65,5 @@
             <xacro:wheel_dimensions />
         </collision>
+        <xacro:cylinder_inertia name="front_left_wheel" radius="${wheel_diameter / 2}" height="${wheel_width}" mass="${wheel_mass}" />
     </link>
     <joint name="front_left_wheel_joint" type="continuous">
@@ -71,4 +80,5 @@
             <xacro:wheel_dimensions />
         </collision>
+        <xacro:cylinder_inertia name="front_right_wheel" radius="${wheel_diameter / 2}" height="${wheel_width}" mass="${wheel_mass}" />
     </link>
     <joint name="front_right_wheel_joint" type="continuous">
@@ -85,4 +95,5 @@
             <xacro:wheel_dimensions />
         </collision>
+        <xacro:cylinder_inertia name="rear_left_wheel" radius="${wheel_diameter / 2}" height="${wheel_width}" mass="${wheel_mass}" />
     </link>
     <joint name="rear_left_wheel_joint" type="continuous">
@@ -99,4 +110,5 @@
             <xacro:wheel_dimensions />
         </collision>
+        <xacro:cylinder_inertia name="rear_right_wheel" radius="${wheel_diameter / 2}" height="${wheel_width}" mass="${wheel_mass}" />
     </link>
     <joint name="rear_right_wheel_joint" type="continuous">

Commit message: rookie in sim, commandable, can receive sensor data; BIG TODO: fix the TF frames for the wheels

File: workspace/src/rookie_description/urdf/rookie.urdf.xacro (robot description, xacro)
@@ -43,4 +43,5 @@
                  ${-(base_height / 2) - ground_clearance + (wheel_diameter / 2)}"
             rpy="0.0 0.0 ${yaw}"/>
+        <axis xyz="0 1 0" />
     </xacro:macro>
     <!-- /Macros -->

File: workspace/src/rookie_description/urdf/rookie_gazebo.xacro (robot description, xacro)
@@ -5,6 +5,8 @@
         <!-- plugin type "imu" -->
         <plugin filename="gz-sim-imu-system" name="gz::sim::systems::Imu" />
-        <!-- LiDAR ('gpu_lidar') plugin, Camera ('camera') -->
-        <plugin filename="gz-sim-sensors-system" name="gz::sim::systems::Sensors" />
+        <!-- LiDAR ('gpu_lidar'), Camera ('camera') -->
+        <plugin filename="gz-sim-sensors-system" name="gz::sim::systems::Sensors">
+            <render_engine>ogre2</render_engine>
+        </plugin>
     </gazebo>
     <!-- "Global" sensors, not explicitly attached to any link -->
@@ -21,5 +23,12 @@
             <odom_publish_frequency>50</odom_publish_frequency>
             <frame_id>odom</frame_id>
-            <topic>cmd_vel</topic>
+            <!-- Internal gazebo topic, NOT ROS topic -->
+            <topic>/model/rookie/cmd_vel</topic>
+        </plugin>
+        <!-- Joint state publishing -->
+        <plugin filename="gz-sim-joint-state-publisher-system" name="gz::sim::systems::JointStatePublisher">
+            <!-- Internal gazebo topic, NOT ROS topic -->
+            <topic>/model/rookie/state</topic>
+            <update_rate>50</update_rate>
         </plugin>
     </gazebo>
@@ -31,5 +40,6 @@
             <update_rate>20</update_rate>
             <visualize>false</visualize>
-            <topic>imu</topic>
+            <!-- Internal gazebo topic, NOT ROS topic -->
+            <topic>/model/rookie/imu</topic>
         </sensor>
     </gazebo>
@@ -38,7 +48,7 @@
         <sensor name="lidar_slamtec_c1_sensor" type="gpu_lidar">
             <pose relative_to='lidar_joint'>0 0 0 0 0 0</pose>
-            <always_on>1</always_on>
-            <visualize>true</visualize>
-            <topic>lidar</topic>
+            <!-- Internal gazebo topic, NOT ROS topic -->
+            <topic>/model/rookie/lidar</topic>
+            <frame_id>lidar_slamtec_c1</frame_id>
             <update_rate>10</update_rate>
             <ray>
@@ -63,4 +73,6 @@
                 </range>
             </ray>
+            <always_on>1</always_on>
+            <visualize>true</visualize>
         </sensor>
     </gazebo>
@@ -81,5 +93,6 @@
           <update_rate>30</update_rate>
           <visualize>true</visualize>
-          <topic>camera</topic>
+          <!-- Internal gazebo topic, NOT ROS topic -->
+          <topic>/model/rookie/camera</topic>
         </sensor>
     </gazebo>

Commit message: fixed tf tree for wheels, robot is drivable

File: workspace/src/rookie_description/urdf/rookie.urdf.xacro (robot description, xacro)
@@ -4,5 +4,8 @@
     <xacro:property name="wheel_base" value="0.129" />
     <!-- Track width: center to center distance between left and right wheels -->
-    <xacro:property name="track_width" value="0.204" />
+    <!-- <xacro:property name="track_width" value="0.204" /> -->
+    <!-- TODO: need to widen the robot (or make the wheel_base shorter) so that it can
+         actually turn in place. -->
+    <xacro:property name="track_width" value="${0.204 + .02}" />
     <!-- Ground clearance: distance from bottom of chassis to the ground -->
     <xacro:property name="ground_clearance" value="0.020" /> <!-- approximate -->
@@ -15,7 +18,12 @@
     <xacro:property name="wheel_width" value="0.02032" />
     <xacro:property name="wheel_diameter" value="0.098425" /> <!-- == 3 7/8" -->
-    <!-- wheel spacing: clearance between wheel and body -->
-    <xacro:property name="wheel_spacing" value="0.00546" />
+    <!-- clearance between wheel and body -->
+    <xacro:property name="wheel_clearance" value="0.00546" />
     <xacro:property name="wheel_mass" value="0.0992233" />
+    <!-- The spacing between left and right wheels, made complicated by the fact that within
+         this URDF, the coordinates of the wheels start at the EDGE, not the CENTER;
+         so, this is edge-to-edge distance, rather than center-to-center -->
+    <xacro:property name="left_right_wheel_spacing" value="${track_width - (wheel_width * 2)}" />
+    <xacro:property name="drive_motor_torque_kg_cm" value="5" />
     <!-- Rather than deal with whatever URDF/SDF package-finding weirdness Gazebo has going on,
          just get our mesh paths directly here so we can use them later.-->
@@ -23,6 +31,6 @@
     <!-- Macros -->
     <xacro:include filename="$(find rookie_description)/urdf/macros.xacro" />
-    <xacro:macro name="wheel_dimensions">
-        <origin xyz="0 ${-1 * wheel_width / 2} 0" rpy="1.570796327 0 0"/>
+    <xacro:macro name="wheel_dimensions" params="mirror_y">
+        <origin xyz="0 ${mirror_y * wheel_width / 2} 0" rpy="1.570796327 0 0"/>
         <geometry>
             <cylinder length="${wheel_width}" radius="${wheel_diameter / 2}" />
@@ -32,15 +40,9 @@
         <parent link="base_link" />
         <child link="${wheel_name}" />
-        <xacro:if value="${mirror_y == -1}">
-            <xacro:property name="yaw" value="3.14159" />
-        </xacro:if>
-        <xacro:unless value="${mirror_y == -1}">
-            <xacro:property name="yaw" value="0" />
-        </xacro:unless>
         <origin
             xyz="${(wheel_base / 2) * mirror_x}
-                 ${((track_width / 2) + wheel_spacing - (wheel_width / 2)) * mirror_y}
+                 ${((left_right_wheel_spacing / 2) + wheel_clearance - ((mirror_y * wheel_width) / 2)) * mirror_y}
                  ${-(base_height / 2) - ground_clearance + (wheel_diameter / 2)}"
-            rpy="0.0 0.0 ${yaw}"/>
+            rpy="0.0 0.0 0.0"/>
         <axis xyz="0 1 0" />
     </xacro:macro>
@@ -61,5 +63,5 @@
     <link name="front_left_wheel">
         <visual>
-            <origin rpy="0.0 0.0 0.0" xyz="0.0 0.0 0.0" />
+            <origin rpy="0.0 0.0 3.14159" xyz="0.0 0.0 0.0" />
             <geometry>
                 <mesh filename="${mesh_directory}/Banebots_T81_Wheel.dae"/>
@@ -67,5 +69,5 @@
         </visual>
         <collision>
-            <xacro:wheel_dimensions />
+            <xacro:wheel_dimensions mirror_y="-1" />
         </collision>
         <xacro:cylinder_inertia name="front_left_wheel" radius="${wheel_diameter / 2}" height="${wheel_width}" mass="${wheel_mass}" />
@@ -74,7 +76,7 @@
         <xacro:wheel_joint wheel_name="front_left_wheel" mirror_x="1" mirror_y="1" />
     </joint>
-    <link name="front_right_wheel">
+    <link name="rear_left_wheel">
         <visual>
-            <origin rpy="0.0 0.0 0.0" xyz="0.0 0.0 0.0" />
+            <origin rpy="0.0 0.0 3.14159" xyz="0.0 0.0 0.0" />
             <geometry>
                 <mesh filename="${mesh_directory}/Banebots_T81_Wheel.dae"/>
@@ -82,5 +84,20 @@
         </visual>
         <collision>
-            <xacro:wheel_dimensions />
+            <xacro:wheel_dimensions mirror_y="-1" />
+        </collision>
+        <xacro:cylinder_inertia name="rear_left_wheel" radius="${wheel_diameter / 2}" height="${wheel_width}" mass="${wheel_mass}" />
+    </link>
+    <joint name="rear_left_wheel_joint" type="continuous">
+        <xacro:wheel_joint wheel_name="rear_left_wheel" mirror_x="-1" mirror_y="1" />
+    </joint>
+    <link name="front_right_wheel">
+        <visual>
+            <origin rpy="0.0 0.0 3.14159" xyz="0.0 0.0 0.0" />
+            <geometry>
+                <mesh filename="${mesh_directory}/Banebots_T81_Wheel.dae"/>
+            </geometry>
+        </visual>
+        <collision>
+            <xacro:wheel_dimensions mirror_y="1"/>
         </collision>
         <xacro:cylinder_inertia name="front_right_wheel" radius="${wheel_diameter / 2}" height="${wheel_width}" mass="${wheel_mass}" />
@@ -89,7 +106,7 @@
         <xacro:wheel_joint wheel_name="front_right_wheel" mirror_x="1" mirror_y="-1" />
     </joint>
-    <link name="rear_left_wheel">
+    <link name="rear_right_wheel">
         <visual>
-            <origin rpy="0.0 0.0 0.0" xyz="0.0 0.0 0.0" />
+            <origin rpy="0.0 0.0 3.14159" xyz="0.0 0.0 0.0" />
             <geometry>
                 <mesh filename="${mesh_directory}/Banebots_T81_Wheel.dae"/>
@@ -97,20 +114,5 @@
         </visual>
         <collision>
-            <xacro:wheel_dimensions />
-        </collision>
-        <xacro:cylinder_inertia name="rear_left_wheel" radius="${wheel_diameter / 2}" height="${wheel_width}" mass="${wheel_mass}" />
-    </link>
-    <joint name="rear_left_wheel_joint" type="continuous">
-        <xacro:wheel_joint wheel_name="rear_left_wheel" mirror_x="-1" mirror_y="1" />
-    </joint>
-    <link name="rear_right_wheel">
-        <visual>
-            <origin rpy="0.0 0.0 0.0" xyz="0.0 0.0 0.0" />
-            <geometry>
-                <mesh filename="${mesh_directory}/Banebots_T81_Wheel.dae"/>
-            </geometry>
-        </visual>
-        <collision>
-            <xacro:wheel_dimensions />
+            <xacro:wheel_dimensions mirror_y="1"/>
         </collision>
         <xacro:cylinder_inertia name="rear_right_wheel" radius="${wheel_diameter / 2}" height="${wheel_width}" mass="${wheel_mass}" />

File: workspace/src/rookie_description/urdf/rookie_gazebo.xacro (robot description, xacro)
@@ -25,4 +25,6 @@
             <!-- Internal gazebo topic, NOT ROS topic -->
             <topic>/model/rookie/cmd_vel</topic>
+            <!-- TODO: I have no idea if this param is even doing anything...-->
+            <max_wheel_torque>${drive_motor_torque_kg_cm / 2}</max_wheel_torque>
         </plugin>
         <!-- Joint state publishing -->
