Commit message: checkpoint: working odom->base_link transform and EKF-ed odometry in simulation

File: workspace/src/rookie_description/urdf/rookie.gazebo.xacro (robot description, xacro)
@@ -38,12 +38,15 @@
     </gazebo>
     <!-- Sensors attached to the base_link -->
-    <gazebo reference="base_link">
+    <!-- <gazebo reference="base_link"> -->
+    <gazebo reference="imu">
+        <!-- <plugin filename="gz-sim-imu-system" name="gz::sim::systems::Imu" /> -->
         <!-- IMU plugin -->
         <sensor name="imu_sensor" type="imu">
+            <!-- Internal gazebo topic, NOT ROS topic -->
+            <topic>/model/rookie/imu</topic>
+            <frame_id>imu</frame_id>
             <always_on>1</always_on>
             <update_rate>20</update_rate>
             <visualize>false</visualize>
-            <!-- Internal gazebo topic, NOT ROS topic -->
-            <topic>/model/rookie/imu</topic>
         </sensor>
     </gazebo>
@@ -83,20 +86,20 @@
     <gazebo reference="camera">
         <sensor name="camera_sensor" type="camera">
-          <camera>
-            <horizontal_fov>1.047</horizontal_fov>
-            <image>
-              <width>320</width>
-              <height>240</height>
-            </image>
-            <clip>
-              <near>0.1</near>
-              <far>100</far>
-            </clip>
-          </camera>
-          <always_on>1</always_on>
-          <update_rate>30</update_rate>
-          <visualize>true</visualize>
-          <!-- Internal gazebo topic, NOT ROS topic -->
-          <topic>/model/rookie/camera</topic>
+            <camera>
+                <horizontal_fov>1.047</horizontal_fov>
+                <image>
+                    <width>320</width>
+                    <height>240</height>
+                </image>
+                <clip>
+                    <near>0.1</near>
+                    <far>100</far>
+                </clip>
+            </camera>
+            <always_on>1</always_on>
+            <update_rate>30</update_rate>
+            <visualize>true</visualize>
+            <!-- Internal gazebo topic, NOT ROS topic -->
+            <topic>/model/rookie/camera</topic>
         </sensor>
     </gazebo>

File: workspace/src/rookie_description/urdf/rookie.urdf.xacro (robot description, xacro)
@@ -25,4 +25,5 @@
          so, this is edge-to-edge distance, rather than center-to-center -->
     <xacro:property name="left_right_wheel_spacing" value="${track_width - (wheel_width * 2)}" />
+    <!-- Motor params -->
     <xacro:property name="drive_motor_torque_kg_cm" value="5" />
     <!-- Rather than deal with whatever URDF/SDF package-finding weirdness Gazebo has going on,
@@ -156,5 +157,20 @@
             rpy="0.0 0.0 0"/>
     </joint>
+    <link name="imu" type="fixed">
+        <static>true</static>
+        <visual name='visual'>
+            <geometry>
+                <box size="0.01 0.01 0.01" />
+            </geometry>
+        </visual>
+    </link>
+    <joint name="imu_joint" type="fixed">
+        <parent link="base_link" />
+        <child link="imu" />
+        <origin
+            xyz="0.0 0.0 0.0"
+            rpy="0.0 0.0 0"/>
+    </joint>
     <!-- Gazebo-specific -->
-    <xacro:include filename="$(find rookie_description)/urdf/rookie_gazebo.xacro" />
+    <xacro:include filename="$(find rookie_description)/urdf/rookie.gazebo.xacro" />
 </robot>
